File: n2-etoile-0v.kicad_pcb (KiCad board)
At the start: 2 copper layers, 110 x 68 mm, 21 parts, among them J1 BP J31 (WR-MPC3 2x2), J2 BA1 J1 (WR-MPC3 2x2), J3 BA1 J2 (WR-MPC3 2x2), J4 BA2 J1 (WR-MPC3 2x2), J5 BA2 J2 (WR-MPC3 2x2), J6 BA3 J1 (WR-MPC3 2x2), J7 BA3 J2 (WR-MPC3 2x2), J8 Queue de cochon AWG20 -> J31-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

Commit message: feat(n2): module ESP32 espion/alarme, schéma et PCB routé rév. B (essensys-hub/essensys-feature-lifecycle#28)
- Schéma : ESP32-C3-MINI-1, isolateur ISO7720 2/0 (bus -> module seulement), 1 kΩ série,
  cavalier JP4, LDO LP2950 côté bus, RTC RV-3028 + supercondensateur, TCA9534.
- Mesures : +15 V amont/aval des PTC (÷16), écart de 0 V (TLV9064, G = 0,249),
  4 x MCP3428, latch surtension (2 x LM339 + 74HC74, réarmement GPIO7).
- Alimentation : PTC propre, SS14, SMAJ16A, AP63205 15->5 V, AP2112 3,3 V,
  chargeur LiFePO4 CN3058E 3,6 V 200 mA avec CTN, power-path SS14/AO3401A, 18650.
- Alarme : 4 boucles équilibrées protégées, clé ARM, sirène 12 V (MT3608 + BTS4140N).
- PCB 235 x 68 mm : zone bus (0 V) / zone module (GND) séparées, liaison unique NT1,
  aucune liaison au PE, zone sans cuivre sous l'antenne, sérigraphie TBTS conservée.
- Routeur maillé déterministe (scripts/autoroute.py) ; ERC 0, DRC 0 avec parité schéma.
- README : tolérances des chaînes de mesure (tâche 1.2), budget de consommation, GPIO.

Feature: n2-esp32-spy-alarm-2026-10-008
Co-Authored-By: Claude Opus 5.5 <noreply@anthropic.com>
Parts:
- added BT1: LiFePO4 18650 3,2 V 1,5 Ah, Battery:BatteryHolder_Keystone_1042_1x18650, F.Cu at (175.0, 56.6)
- added C1: 100n, Capacitor_SMD:C_0603_1608Metric, F.Cu at (104.5, 9.50)
- added C10: 10u, Capacitor_SMD:C_0805_2012Metric, F.Cu at (120.0, 38.0)
- added C11: 1u, Capacitor_SMD:C_0603_1608Metric, F.Cu at (119.5, 55.0)
- added C12: 10u, Capacitor_SMD:C_0805_2012Metric, F.Cu at (124.0, 55.0)
- added C13: 1u, Capacitor_SMD:C_0603_1608Metric, F.Cu at (120.5, 43.0)
- added C14: 10u, Capacitor_SMD:C_0805_2012Metric, F.Cu at (129.5, 43.0)
- added C15: 1n, Capacitor_SMD:C_0603_1608Metric, F.Cu at (119.5, 61.5)
- added C16: 10u, Capacitor_SMD:C_0805_2012Metric, F.Cu at (118.5, 8.20)
- added C17: 100n, Capacitor_SMD:C_0603_1608Metric, F.Cu at (118.5, 11.5)
- added C18: 1u, Capacitor_SMD:C_0603_1608Metric, F.Cu at (116.0, 17.2)
- added C19: 100n, Capacitor_SMD:C_0603_1608Metric, F.Cu at (158.3, 13.5)
- added C2: 100n, Capacitor_SMD:C_0603_1608Metric, F.Cu at (116.0, 13.0)
- added C20: 11m 3,3V, Capacitor_SMD:C_1210_3225Metric, F.Cu at (161.2, 15.2)
- added C21: 100n, Capacitor_SMD:C_0603_1608Metric, F.Cu at (147.7, 22.5)
- added C3: 1u 50V, Capacitor_SMD:C_0805_2012Metric, F.Cu at (105.0, 18.0)
- added C30: 100p, Capacitor_SMD:C_0603_1608Metric, F.Cu at (141.8, 38.0)
- added C31: 1n, Capacitor_SMD:C_0603_1608Metric, F.Cu at (144.4, 34.0)
- added C32: 1n, Capacitor_SMD:C_0603_1608Metric, F.Cu at (144.4, 41.9)
- added C33: 1n, Capacitor_SMD:C_0603_1608Metric, F.Cu at (147.1, 38.0)
- added C34: 1n, Capacitor_SMD:C_0603_1608Metric, F.Cu at (158.3, 38.0)
- added C35: 1n, Capacitor_SMD:C_0603_1608Metric, F.Cu at (161.0, 34.0)
- added C36: 1n, Capacitor_SMD:C_0603_1608Metric, F.Cu at (161.0, 41.9)
- added C4: 2u2, Capacitor_SMD:C_0603_1608Metric, F.Cu at (104.5, 12.5)
- added C40: 100n, Capacitor_SMD:C_0603_1608Metric, F.Cu at (191.4, 34.0)
- added C41: 100n, Capacitor_SMD:C_0603_1608Metric, F.Cu at (196.7, 38.0)
- added C42: 100n, Capacitor_SMD:C_0603_1608Metric, F.Cu at (147.1, 41.9)
- added C43: 100n, Capacitor_SMD:C_0603_1608Metric, F.Cu at (163.6, 34.0)
- added C44: 100n, Capacitor_SMD:C_0603_1608Metric, F.Cu at (189.5, 27.5)
- added C45: 100n, Capacitor_SMD:C_0603_1608Metric, F.Cu at (207.9, 34.0)
- added C46: 100n, Capacitor_SMD:C_0603_1608Metric, F.Cu at (221.5, 28.0)
- added C47: 100n, Capacitor_SMD:C_0603_1608Metric, F.Cu at (232.0, 28.0)
- added C48: 100n, Capacitor_SMD:C_0603_1608Metric, F.Cu at (216.0, 40.6)
- added C5: 10u 35V, Capacitor_SMD:C_1206_3216Metric, F.Cu at (128.0, 28.0)
- added C51: 10n, Capacitor_SMD:C_0603_1608Metric, F.Cu at (188.4, 18.6)
- added C52: 10n, Capacitor_SMD:C_0603_1608Metric, F.Cu at (181.4, 18.6)
- added C53: 10n, Capacitor_SMD:C_0603_1608Metric, F.Cu at (174.4, 18.6)
- added C54: 10n, Capacitor_SMD:C_0603_1608Metric, F.Cu at (167.4, 18.6)
- added C55: 22u 25V, Capacitor_SMD:C_1206_3216Metric, F.Cu at (223.0, 21.3)
- added C56: 10u, Capacitor_SMD:C_0805_2012Metric, F.Cu at (220.5, 20.7)
- added C57: 1n, Capacitor_SMD:C_0603_1608Metric, F.Cu at (207.8, 25.5)
- added C6: 100n 50V, Capacitor_SMD:C_0603_1608Metric, F.Cu at (128.0, 32.5)
- added C7: 100n, Capacitor_SMD:C_0603_1608Metric, F.Cu at (132.5, 26.5)
- added C8: 22u 10V, Capacitor_SMD:C_1206_3216Metric, F.Cu at (138.0, 35.0)
- added C9: 22u 10V, Capacitor_SMD:C_1206_3216Metric, F.Cu at (138.0, 38.0)
- added D11: SMF5V0A, Diode_SMD:D_SMF, F.Cu at (188.2, 14.2)
- added D12: SMF5V0A, Diode_SMD:D_SMF, F.Cu at (181.2, 14.2)
- added D13: SMF5V0A, Diode_SMD:D_SMF, F.Cu at (174.2, 14.2)
- added D14: SMF5V0A, Diode_SMD:D_SMF, F.Cu at (167.2, 14.2)
- added D15: SMF5V0A, Diode_SMD:D_SMF, F.Cu at (205.8, 14.2)
- added D16: SMAJ16A, Diode_SMD:D_SMA, F.Cu at (200.5, 15.5)
- added D4: SS14, Diode_SMD:D_SMA, F.Cu at (119.8, 30.0)
- added D5: SMAJ16A, Diode_SMD:D_SMA, F.Cu at (124.2, 30.0)
- added D6: SS14, Diode_SMD:D_SMA, F.Cu at (131.0, 38.0)
- added D7: SS14, Diode_SMD:D_SMA, F.Cu at (215.5, 20.8)
- added F4: PTC 0,2 A 1812, Fuse:Fuse_1812_4532Metric, F.Cu at (115.3, 30.0)
- added F5: PTC 1,5 A 1812, Fuse:Fuse_1812_4532Metric, F.Cu at (127.0, 49.0)
- added H5: M3 isolé, MountingHole:MountingHole_3.2mm_M3, F.Cu at (231.0, 4.00)
- added H6: M3 isolé, MountingHole:MountingHole_3.2mm_M3, F.Cu at (231.0, 64.0)
- added J10: Boucles Z1-Z4, TerminalBlock_Phoenix:TerminalBlock_Phoenix_PT-1,5-8-3.5-H_1x08_P3.50mm_Horizontal, F.Cu at (190.0, 6.50)
- added J11: Clé ARM / sirène 12 V, TerminalBlock_Phoenix:TerminalBlock_Phoenix_PT-1,5-4-3.5-H_1x04_P3.50mm_Horizontal, F.Cu at (207.5, 6.50)
- added J9: Débogage UART/USB, Connector_PinHeader_2.54mm:PinHeader_2x04_P2.54mm_Vertical, F.Cu at (138.0, 9.00)
- added JP4: Cavalier d'écoute (2 shunts), Connector_PinHeader_2.54mm:PinHeader_2x02_P2.54mm_Vertical, F.Cu at (93.0, 9.50)
- added L1: 4,7u, Inductor_SMD:L_Taiyo-Yuden_NR-40xx, F.Cu at (138.0, 30.0)
- added L2: 22u, Inductor_SMD:L_Taiyo-Yuden_NR-50xx, F.Cu at (221.3, 14.3)
- added LED1: LED verte (état), LED_SMD:LED_0603_1608Metric, F.Cu at (140.0, 20.0)
- added LED2: LED rouge (alarme), LED_SMD:LED_0603_1608Metric, F.Cu at (165.7, 25.9)
- added NT1: NetTie 0V-GND, NetTie:NetTie-2_SMD_Pad2.0mm, F.Cu at (111.0, 37.0)
- added Q1: AO3401A, Package_TO_SOT_SMD:SOT-23, F.Cu at (125.0, 38.0)
- added R1: 1k, Resistor_SMD:R_0603_1608Metric, F.Cu at (100.0, 9.50)
- added R10: 100k, Resistor_SMD:R_0603_1608Metric, F.Cu at (115.0, 63.0)
- added R11: 10k, Resistor_SMD:R_0603_1608Metric, F.Cu at (118.5, 15.9)
- added R12: 10k, Resistor_SMD:R_0603_1608Metric, F.Cu at (118.5, 19.0)
- added R13: 10k, Resistor_SMD:R_0603_1608Metric, F.Cu at (134.0, 20.0)
- added R14: 10k, Resistor_SMD:R_0603_1608Metric, F.Cu at (136.0, 20.0)
- added R15: 10k, Resistor_SMD:R_0603_1608Metric, F.Cu at (138.0, 20.0)
- added R16: 1k, Resistor_SMD:R_0603_1608Metric, F.Cu at (142.0, 20.0)
- added R17: 4k7, Resistor_SMD:R_0603_1608Metric, F.Cu at (145.8, 22.5)
- added R18: 4k7, Resistor_SMD:R_0603_1608Metric, F.Cu at (145.8, 25.9)
- added R19: 10k, Resistor_SMD:R_0603_1608Metric, F.Cu at (161.9, 22.5)
- added R2: 1k, Resistor_SMD:R_0603_1608Metric, F.Cu at (100.0, 12.0)
- added R20: 10k, Resistor_SMD:R_0603_1608Metric, F.Cu at (161.9, 25.9)
- added R21: 10k, Resistor_SMD:R_0603_1608Metric, F.Cu at (163.8, 22.5)
- added R22: 1k, Resistor_SMD:R_0603_1608Metric, F.Cu at (165.7, 22.5)
- added R23: 10k, Resistor_SMD:R_0603_1608Metric, F.Cu at (163.8, 25.9)
- added R3: 100, Resistor_SMD:R_1206_3216Metric, F.Cu at (95.0, 19.0)
- added R30: 150k, Resistor_SMD:R_0805_2012Metric, F.Cu at (104.0, 23.0)
- added R31: 150k, Resistor_SMD:R_0805_2012Metric, F.Cu at (36.0, 38.5)
- added R32: 150k, Resistor_SMD:R_0805_2012Metric, F.Cu at (64.0, 38.5)
- added R33: 150k, Resistor_SMD:R_0805_2012Metric, F.Cu at (92.0, 38.5)
- added R34: 150k, Resistor_SMD:R_0805_2012Metric, F.Cu at (40.0, 44.5)
- added R35: 150k, Resistor_SMD:R_0805_2012Metric, F.Cu at (68.0, 44.5)
- added R36: 150k, Resistor_SMD:R_0805_2012Metric, F.Cu at (96.0, 44.5)
- added R4: 100k, Resistor_SMD:R_0603_1608Metric, F.Cu at (133.0, 34.0)
- added R40: 10k, Resistor_SMD:R_0603_1608Metric, F.Cu at (141.8, 34.0)
- added R41: 10k, Resistor_SMD:R_0603_1608Metric, F.Cu at (141.8, 41.9)
- added R42: 10k, Resistor_SMD:R_0603_1608Metric, F.Cu at (144.4, 38.0)
- added R43: 10k, Resistor_SMD:R_0603_1608Metric, F.Cu at (147.1, 34.0)
- added R44: 10k, Resistor_SMD:R_0603_1608Metric, F.Cu at (158.3, 34.0)
- added R45: 10k, Resistor_SMD:R_0603_1608Metric, F.Cu at (158.3, 41.9)
- added R46: 10k, Resistor_SMD:R_0603_1608Metric, F.Cu at (161.0, 38.0)
- added R5: 9k1, Resistor_SMD:R_0603_1608Metric, F.Cu at (115.0, 55.0)
- added R51: 100k, Resistor_SMD:R_1206_3216Metric, F.Cu at (24.0, 61.0)
- added R52: 100k, Resistor_SMD:R_1206_3216Metric, F.Cu at (52.0, 61.0)
- added R53: 100k, Resistor_SMD:R_1206_3216Metric, F.Cu at (80.0, 61.0)
- added R54: 100k, Resistor_SMD:R_1206_3216Metric, F.Cu at (4.50, 46.0)
- added R55: 100k, Resistor_SMD:R_1206_3216Metric, F.Cu at (4.50, 49.0)
- added R56: 100k, Resistor_SMD:R_1206_3216Metric, F.Cu at (4.50, 52.0)
- added R57: 24k9, Resistor_SMD:R_0603_1608Metric, F.Cu at (174.9, 34.0)
- added R58: 24k9, Resistor_SMD:R_0603_1608Metric, F.Cu at (177.5, 34.0)
- added R59: 24k9, Resistor_SMD:R_0603_1608Metric, F.Cu at (180.2, 34.0)
- added R6: 6k2, Resistor_SMD:R_0603_1608Metric, F.Cu at (115.0, 57.5)
- added R60: 24k9, Resistor_SMD:R_0603_1608Metric, F.Cu at (174.9, 38.0)
- added R61: 24k9, Resistor_SMD:R_0603_1608Metric, F.Cu at (177.5, 38.0)
- added R62: 24k9, Resistor_SMD:R_0603_1608Metric, F.Cu at (180.2, 38.0)
- added R63: 20k5, Resistor_SMD:R_0603_1608Metric, F.Cu at (191.4, 38.0)
- added R64: 2k49, Resistor_SMD:R_0603_1608Metric, F.Cu at (194.0, 34.0)
- added R65: 2k49, Resistor_SMD:R_0603_1608Metric, F.Cu at (194.0, 38.0)
- added R66: 7k5, Resistor_SMD:R_0603_1608Metric, F.Cu at (196.7, 34.0)
- added R67: 10k, Resistor_SMD:R_0603_1608Metric, F.Cu at (221.5, 32.2)
- added R68: 10k, Resistor_SMD:R_0603_1608Metric, F.Cu at (232.0, 32.2)
- added R69: 10k, Resistor_SMD:R_0603_1608Metric, F.Cu at (227.0, 40.6)
- added R7: 10k, Resistor_SMD:R_0603_1608Metric, F.Cu at (134.0, 42.5)
- added R71: 1k, Resistor_SMD:R_0805_2012Metric, F.Cu at (191.6, 14.2)
- added R72: 1k, Resistor_SMD:R_0805_2012Metric, F.Cu at (184.6, 14.2)
- added R73: 1k, Resistor_SMD:R_0805_2012Metric, F.Cu at (177.6, 14.2)
- added R74: 1k, Resistor_SMD:R_0805_2012Metric, F.Cu at (170.6, 14.2)
- added R75: 10k, Resistor_SMD:R_0603_1608Metric, F.Cu at (191.6, 18.6)
- added R76: 10k, Resistor_SMD:R_0603_1608Metric, F.Cu at (184.6, 18.6)
- added R77: 10k, Resistor_SMD:R_0603_1608Metric, F.Cu at (177.6, 18.6)
- added R78: 10k, Resistor_SMD:R_0603_1608Metric, F.Cu at (170.6, 18.6)
- added R79: 1k, Resistor_SMD:R_0805_2012Metric, F.Cu at (209.1, 14.2)
- added R8: 20k, Resistor_SMD:R_0603_1608Metric, F.Cu at (134.0, 44.5)
- added R80: 10k, Resistor_SMD:R_0603_1608Metric, F.Cu at (209.1, 18.6)
- added R81: 191k, Resistor_SMD:R_0603_1608Metric, F.Cu at (217.3, 13.0)
- added R82: 10k, Resistor_SMD:R_0603_1608Metric, F.Cu at (217.3, 16.4)
- added R83: 100k, Resistor_SMD:R_0603_1608Metric, F.Cu at (204.0, 25.5)
- added R84: 100k, Resistor_SMD:R_0603_1608Metric, F.Cu at (205.9, 25.5)
- added R85: 10k, Resistor_SMD:R_0603_1608Metric, F.Cu at (205.9, 28.9)
- added R9: 100k, Resistor_SMD:R_0603_1608Metric, F.Cu at (115.0, 60.5)
- added SW1: BOOT / service, Button_Switch_SMD:SW_SPST_PTS645Sx43SMTR92, F.Cu at (148.0, 12.0)
- added TH1: CTN 10k B3435, Resistor_SMD:R_0603_1608Metric, F.Cu at (128.0, 62.0)
- added U1: ISO7720D, Package_SO:SOIC-8_3.9x4.9mm_P1.27mm, F.Cu at (111.0, 13.0)
- added U10: MCP3428-E/SL, Package_SO:SOIC-14_3.9x8.7mm_P1.27mm, F.Cu at (152.7, 37.1)
- added U11: MCP3428-E/SL, Package_SO:SOIC-14_3.9x8.7mm_P1.27mm, F.Cu at (169.2, 37.1)
- added U12: MCP3428-E/SL, Package_SO:SOIC-14_3.9x8.7mm_P1.27mm, F.Cu at (184.5, 27.5)
- added U13: MCP3428-E/SL, Package_SO:SOIC-14_3.9x8.7mm_P1.27mm, F.Cu at (202.3, 37.1)
- added U14: LM339, Package_SO:SOIC-14_3.9x8.7mm_P1.27mm, F.Cu at (216.5, 31.0)
- added U15: LM339, Package_SO:SOIC-14_3.9x8.7mm_P1.27mm, F.Cu at (227.0, 31.0)
- added U16: 74HC74, Package_SO:SOIC-14_3.9x8.7mm_P1.27mm, F.Cu at (221.5, 40.6)
- added U17: MT3608, Package_TO_SOT_SMD:SOT-23-6, F.Cu at (214.1, 13.2)
- added U18: BTS4140N, Package_TO_SOT_SMD:SOT-223, F.Cu at (198.4, 27.6)
- added U2: LP2950-5.0, Package_TO_SOT_THT:TO-92_Inline, F.Cu at (99.0, 18.0)
- added U3: AP63205WU, Package_TO_SOT_SMD:TSOT-23-6, F.Cu at (132.5, 30.0)
- added U4: CN3058E, Package_SO:SOIC-8-1EP_3.9x4.9mm_P1.27mm_EP2.41x3.3mm, F.Cu at (118.0, 50.0)
- added U5: AP2112K-3.3, Package_TO_SOT_SMD:SOT-23-5, F.Cu at (125.0, 43.0)
- added U6: ESP32-C3-MINI-1, RF_Module:ESP32-C6-MINI-1, F.Cu at (127.0, 12.0)
- added U7: RV-3028-C7, Package_SON:MicroCrystal_C7_SON-8_1.5x3.2mm_P0.9mm, F.Cu at (155.5, 13.5)
- added U8: TCA9534DW, Package_SO:SOIC-16W_7.5x10.3mm_P1.27mm, F.Cu at (154.8, 26.4)
- added U9: TLV9064IDR, Package_SO:SOIC-14_3.9x8.7mm_P1.27mm, F.Cu at (185.8, 37.1)
- moved H2 5.00 mm to (101.0, 4.00)
Routing:
- net /3V3: track 0.00 -> 417.9 mm, vias 0 -> 41
- net /GND: track 0.00 -> 359.8 mm, vias 0 -> 348
- net /VBAT: track 0.00 -> 311.9 mm, vias 0 -> 24
- net /I2C_SCL: track 0.00 -> 225.0 mm, vias 0 -> 22
- net /I2C_SDA: track 0.00 -> 198.0 mm, vias 0 -> 21
- net /DA_M3: track 0.00 -> 196.9 mm, vias 0 -> 11
- net /DA_M1: track 0.00 -> 192.4 mm, vias 0 -> 12
- net /DA_M2: track 0.00 -> 191.7 mm, vias 0 -> 12
- net /MEAS_15BP: track 0.00 -> 190.7 mm, vias 0 -> 11
- net /DA_P1: track 0.00 -> 169.2 mm, vias 0 -> 2
- net /DA_P2: track 0.00 -> 155.7 mm, vias 0 -> 11
- net /LATCH_RST: track 0.00 -> 146.5 mm, vias 0 -> 17
- net /MEAS_BA1: track 0.00 -> 141.4 mm, vias 0 -> 4
- net /LATCH_0V: track 0.00 -> 134.6 mm, vias 0 -> 7
- net /MEAS_SW1: track 0.00 -> 131.9 mm, vias 0 -> 3
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- added copper zone on B.Cu, net /GND
- added copper zone on F.Cu, net /GND
Other:
- board size 110 x 68 mm -> 235 x 68 mm
- board text added: "N2 ÉTOILE 0 V rév. B – essensys-i2c-etoile-0v"
- board text added: "ZONE MODULE (GND) – TBTS – AUCUNE LIAISON AU PE"
- board text removed: "N2 ÉTOILE 0 V rév. A – essensys-i2c-etoile-0v"
