File: n2-etoile-0v.kicad_sch (KiCad schematic)
At the start: 17 parts, among them J1 BP J31 (WR-MPC3 2x2), J2 BA1 J1 (WR-MPC3 2x2), J3 BA1 J2 (WR-MPC3 2x2), J4 BA2 J1 (WR-MPC3 2x2), J5 BA2 J2 (WR-MPC3 2x2), J6 BA3 J1 (WR-MPC3 2x2), J7 BA3 J2 (WR-MPC3 2x2), J8 Queue de cochon AWG20 -> J31-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

Commit message: feat(n2): module ESP32 espion/alarme, schéma et PCB routé rév. B (essensys-hub/essensys-feature-lifecycle#28)
- Schéma : ESP32-C3-MINI-1, isolateur ISO7720 2/0 (bus -> module seulement), 1 kΩ série,
  cavalier JP4, LDO LP2950 côté bus, RTC RV-3028 + supercondensateur, TCA9534.
- Mesures : +15 V amont/aval des PTC (÷16), écart de 0 V (TLV9064, G = 0,249),
  4 x MCP3428, latch surtension (2 x LM339 + 74HC74, réarmement GPIO7).
- Alimentation : PTC propre, SS14, SMAJ16A, AP63205 15->5 V, AP2112 3,3 V,
  chargeur LiFePO4 CN3058E 3,6 V 200 mA avec CTN, power-path SS14/AO3401A, 18650.
- Alarme : 4 boucles équilibrées protégées, clé ARM, sirène 12 V (MT3608 + BTS4140N).
- PCB 235 x 68 mm : zone bus (0 V) / zone module (GND) séparées, liaison unique NT1,
  aucune liaison au PE, zone sans cuivre sous l'antenne, sérigraphie TBTS conservée.
- Routeur maillé déterministe (scripts/autoroute.py) ; ERC 0, DRC 0 avec parité schéma.
- README : tolérances des chaînes de mesure (tâche 1.2), budget de consommation, GPIO.

Feature: n2-esp32-spy-alarm-2026-10-008
Co-Authored-By: Claude Opus 5.5 <noreply@anthropic.com>
Parts:
- added BT1: LiFePO4 18650 3,2 V 1,5 Ah, Battery:BatteryHolder_Keystone_1042_1x18650, symbol Device:Battery_Cell
- added C1, C17, C19, C2, C21, C40, C41, C42, C43, C44, C45, C46, C47, C48, C7: 100n, Capacitor_SMD:C_0603_1608Metric, symbol Device:C
- added C10, C12, C14, C16, C56: 10u, Capacitor_SMD:C_0805_2012Metric, symbol Device:C
- added C11, C13, C18: 1u, Capacitor_SMD:C_0603_1608Metric, symbol Device:C
- added C15, C31, C32, C33, C34, C35, C36, C57: 1n, Capacitor_SMD:C_0603_1608Metric, symbol Device:C
- added C20: 11m 3,3V, Capacitor_SMD:C_1210_3225Metric, symbol Device:C
- added C3: 1u 50V, Capacitor_SMD:C_0805_2012Metric, symbol Device:C
- added C30: 100p, Capacitor_SMD:C_0603_1608Metric, symbol Device:C
- added C4: 2u2, Capacitor_SMD:C_0603_1608Metric, symbol Device:C
- added C5: 10u 35V, Capacitor_SMD:C_1206_3216Metric, symbol Device:C
- added C51, C52, C53, C54: 10n, Capacitor_SMD:C_0603_1608Metric, symbol Device:C
- added C55: 22u 25V, Capacitor_SMD:C_1206_3216Metric, symbol Device:C
- added C6: 100n 50V, Capacitor_SMD:C_0603_1608Metric, symbol Device:C
- added C8, C9: 22u 10V, Capacitor_SMD:C_1206_3216Metric, symbol Device:C
- added D11, D12, D13, D14, D15: SMF5V0A, Diode_SMD:D_SMF, symbol Diode:SMF5V0A
- added D16, D5: SMAJ16A, Diode_SMD:D_SMA, symbol Diode:SMAJ16A
- added D4, D6, D7: SS14, Diode_SMD:D_SMA, symbol Diode:SS14
- added F4: PTC 0,2 A 1812, Fuse:Fuse_1812_4532Metric, symbol Device:Polyfuse
- added F5: PTC 1,5 A 1812, Fuse:Fuse_1812_4532Metric, symbol Device:Polyfuse
- added J10: Boucles Z1-Z4, TerminalBlock_Phoenix:TerminalBlock_Phoenix_PT-1,5-8-3.5-H_1x08_P3.50mm_Horizontal, symbol Connector_Generic:Conn_01x08
- added J11: Clé ARM / sirène 12 V, TerminalBlock_Phoenix:TerminalBlock_Phoenix_PT-1,5-4-3.5-H_1x04_P3.50mm_Horizontal, symbol Connector_Generic:Conn_01x04
- added J9: Débogage UART/USB, Connector_PinHeader_2.54mm:PinHeader_2x04_P2.54mm_Vertical, symbol Connector_Generic:Conn_02x04_Odd_Even
- added JP4: Cavalier d'écoute (2 shunts), Connector_PinHeader_2.54mm:PinHeader_2x02_P2.54mm_Vertical, symbol Connector_Generic:Conn_02x02_Odd_Even
- added L1: 4,7u, Inductor_SMD:L_Taiyo-Yuden_NR-40xx, symbol Device:L
- added L2: 22u, Inductor_SMD:L_Taiyo-Yuden_NR-50xx, symbol Device:L
- added LED1: LED verte (état), LED_SMD:LED_0603_1608Metric, symbol Device:LED
- added LED2: LED rouge (alarme), LED_SMD:LED_0603_1608Metric, symbol Device:LED
- added NT1: NetTie 0V-GND, NetTie:NetTie-2_SMD_Pad2.0mm, symbol Device:NetTie_2
- added Q1: AO3401A, Package_TO_SOT_SMD:SOT-23, symbol Transistor_FET:AO3401A
- added R1, R16, R2, R22: 1k, Resistor_SMD:R_0603_1608Metric, symbol Device:R
- added R10, R4, R83, R84, R9: 100k, Resistor_SMD:R_0603_1608Metric, symbol Device:R
- added R11, R12, R13, R14, R15, R19, R20, R21, R23, R40, R41, R42, R43, R44, R45, R46, R67, R68, R69, R7, R75, R76, R77, R78, R80, R82, R85: 10k, Resistor_SMD:R_0603_1608Metric, symbol Device:R
- added R17, R18: 4k7, Resistor_SMD:R_0603_1608Metric, symbol Device:R
- added R3: 100, Resistor_SMD:R_1206_3216Metric, symbol Device:R
- added R30, R31, R32, R33, R34, R35, R36: 150k, Resistor_SMD:R_0805_2012Metric, symbol Device:R
- added R5: 9k1, Resistor_SMD:R_0603_1608Metric, symbol Device:R
- added R51, R52, R53, R54, R55, R56: 100k, Resistor_SMD:R_1206_3216Metric, symbol Device:R
- added R57, R58, R59, R60, R61, R62: 24k9, Resistor_SMD:R_0603_1608Metric, symbol Device:R
- added R6: 6k2, Resistor_SMD:R_0603_1608Metric, symbol Device:R
- added R63: 20k5, Resistor_SMD:R_0603_1608Metric, symbol Device:R
- added R64, R65: 2k49, Resistor_SMD:R_0603_1608Metric, symbol Device:R
- added R66: 7k5, Resistor_SMD:R_0603_1608Metric, symbol Device:R
- added R71, R72, R73, R74, R79: 1k, Resistor_SMD:R_0805_2012Metric, symbol Device:R
- added R8: 20k, Resistor_SMD:R_0603_1608Metric, symbol Device:R
- added R81: 191k, Resistor_SMD:R_0603_1608Metric, symbol Device:R
- added SW1: BOOT / service, Button_Switch_SMD:SW_SPST_PTS645Sx43SMTR92, symbol Switch:SW_Push
- added TH1: CTN 10k B3435, Resistor_SMD:R_0603_1608Metric, symbol Device:Thermistor_NTC
- added U1: ISO7720D, Package_SO:SOIC-8_3.9x4.9mm_P1.27mm, symbol Isolator:ISO7720D
- added U10, U11, U12, U13: MCP3428-E/SL, Package_SO:SOIC-14_3.9x8.7mm_P1.27mm, symbol Analog_ADC:MCP3428x-xSL
- added U14, U15: LM339, Package_SO:SOIC-14_3.9x8.7mm_P1.27mm, symbol Comparator:LM339
- added U16: 74HC74, Package_SO:SOIC-14_3.9x8.7mm_P1.27mm, symbol 74xx:74HC74
- added U17: MT3608, Package_TO_SOT_SMD:SOT-23-6, symbol Regulator_Switching:MT3608
- added U18: BTS4140N, Package_TO_SOT_SMD:SOT-223, symbol Transistor_FET_Other:BTS4140N
- added U2: LP2950-5.0, Package_TO_SOT_THT:TO-92_Inline, symbol Regulator_Linear:LP2950-5.0_TO92
- added U3: AP63205WU, Package_TO_SOT_SMD:TSOT-23-6, symbol Regulator_Switching:AP63205WU
- added U4: CN3058E, Package_SO:SOIC-8-1EP_3.9x4.9mm_P1.27mm_EP2.41x3.3mm, symbol n2:CN3058E
- added U5: AP2112K-3.3, Package_TO_SOT_SMD:SOT-23-5, symbol Regulator_Linear:AP2112K-3.3
- added U6: ESP32-C3-MINI-1, RF_Module:ESP32-C6-MINI-1, symbol n2:ESP32-C3-MINI-1
- added U7: RV-3028-C7, Package_SON:MicroCrystal_C7_SON-8_1.5x3.2mm_P0.9mm, symbol Timer_RTC:RV-3028-C7
- added U8: TCA9534DW, Package_SO:SOIC-16W_7.5x10.3mm_P1.27mm, symbol Interface_Expansion:TCA9534
- added U9: TLV9064IDR, Package_SO:SOIC-14_3.9x8.7mm_P1.27mm, symbol Amplifier_Operational:TLV9064
Connections:
- net +15V_BA1: now also R34.1
- net +15V_BA2: now also R35.1
- net +15V_BA3: now also R36.1
- net +15V_BP: now also F4.1, R3.1, R30.1
- net +15V_SW1: now also R31.1
- net +15V_SW2: now also R32.1
- net +15V_SW3: now also R33.1
- net 0V: now also C1.2, C3.2, C4.2, NT1.1, R51.1, R52.1, R53.1, R54.1, R55.1, R56.1, U1.4 (GND1), U2.2 (GND)
- net SCL_BP: now also JP4.3 (Pin_3)
- net SDA_BP: now also JP4.1 (Pin_1)
- new net +12V_S: C55.1, D7.1 (K), R81.1, U18.2 (V_{bb}), U18.4 (V_{bb})
- new net +15V_ISR: C3.1, R3.2, U2.3 (VI)
- new net +15V_M: C5.1, C6.1, D4.1 (K), D5.1 (A1), U3.2 (EN), U3.3 (IN)
- new net +15V_MF: D4.2 (A), F4.2
- new net +5V: C11.1, C8.1, C9.1, D6.2 (A), L1.2, Q1.1 (G), R4.1, R6.1, R7.1, U3.1 (FB), U4.4 (VIN)
- new net +5V_ISO: C1.1, C4.1, U1.1 (VCC1), U2.1 (VO)
- new net 3V3: C14.1, C16.1, C17.1, C19.1, C2.1, C21.1, C40.1, C42.1, C43.1, C44.1, C45.1, C46.1, C47.1, C48.1, J9.1 (Pin_1), R11.1, R12.1, R13.1, R14.1, R15.1, R16.1, R17.1, R18.1, R19.1, R20.1, R21.1, R22.1, R63.1, R67.1, R68.1, R69.1, R75.1, R76.1, R77.1, R78.1, R80.1, U1.8 (VCC2), U10.6 (V_{DD}), U11.6 (V_{DD}), U11.9 (Adr0), U12.10 (Adr1), U12.6 (V_{DD}), U13.10 (Adr1), U13.6 (V_{DD}), U13.9 (Adr0), U14.3 (V+), U15.3 (V+), U16.14 (VCC), U5.5 (VOUT), U6.3 (3V3), U7.7 (VDD), U8.16 (VDD), U9.4 (V+)
- new net ARM_IN: R79.2, R80.2, U8.9 (P4)
- new net ARM_T: D15.1 (A1), J11.1 (Pin_1), R79.1
- new net BAT_P: BT1.1 (+), F5.1
- new net BOOST_FB: R81.2, R82.1, U17.3 (FB)
- new net BOOST_SW: D7.2 (A), L2.2, U17.1 (SW)
- new net BOOT: J9.6 (Pin_6), R14.2, SW1.1, U6.23 (IO9)
- new net BUCK_BST: C7.1, U3.6 (BST)
- new net BUCK_SW: C7.2, L1.1, U3.5 (SW)
- new net CHG_CHRG: R20.2, U4.7 (~{CHRG}), U8.6 (P2)
- new net CHG_DONE: R21.2, U4.6 (~{DONE}), U8.7 (P3)
- new net CHG_ISET: R5.1, U4.2 (ISET)
- new net CHG_TEMP: R6.2, TH1.1, U4.1 (TEMP)
- new net DA_M1: R54.2, R60.1, U9.2 (-)
- new net DA_M2: R55.2, R61.1, U9.6 (-)
- new net DA_M3: R56.2, R62.1, U9.9 (-)
- new net DA_P1: R51.2, R57.1, U9.3 (+)
- new net DA_P2: R52.2, R58.1, U9.5 (+)
- new net DA_P3: R53.2, R59.1, U9.10 (+)
- new net EN_ESP: C18.1, J9.5 (Pin_5), R11.2, U6.8 (EN)
- new net EXP_INT: R19.2, U6.6 (IO3), U8.13 (~{INT})
- new net EXP_P7: R23.1, U8.12 (P7)
- new net GND: BT1.2 (-), C10.2, C11.2, C12.2, C13.2, C14.2, C15.2, C16.2, C17.2, C18.2, C19.2, C2.2, C20.2, C21.2, C30.2, C31.2, C32.2, C33.2, C34.2, C35.2, C36.2, C40.2, C41.2, C42.2, C43.2, C44.2, C45.2, C46.2, C47.2, C48.2, C5.2, C51.2, C52.2, C53.2, C54.2, C55.2, C56.2, C57.2, C6.2, C8.2, C9.2, D11.2 (A2), D12.2 (A2), D13.2 (A2), D14.2 (A2), D15.2 (A2), D16.2 (A2), D5.2 (A2), J10.2 (Pin_2), J10.4 (Pin_4), J10.6 (Pin_6), J10.8 (Pin_8), J11.2 (Pin_2), J11.4 (Pin_4), J9.2 (Pin_2), NT1.2, R10.2, R23.2, R4.2, R40.2, R41.2, R42.2, R43.2, R44.2, R45.2, R46.2, R5.2, R66.2, R8.2, R82.2, R83.2, R85.2, SW1.2, TH1.2, U1.5 (GND2), U10.10 (Adr1), U10.12 (CH3-), U10.14 (CH4-), U10.2 (CH1-), U10.4 (CH2-), U10.5 (V_{SS}), U10.9 (Adr0), U11.10 (Adr1), U11.12 (CH3-), U11.14 (CH4-), U11.2 (CH1-), U11.4 (CH2-), U11.5 (V_{SS}), U12.12 (CH3-), U12.14 (CH4-), U12.2 (CH1-), U12.4 (CH2-), U12.5 (V_{SS}), U12.9 (Adr0), U13.14 (CH4-), U13.5 (V_{SS}), U14.12 (V-), U15.11 (+), U15.12 (V-), U16.11 (C), U16.12 (D), U16.2 (D), U16.3 (C), U16.7 (GND), U17.2 (GND), U3.4 (GND), U4.3 (GND), U4.9 (GND), U5.2 (GND), U6.1 (GND), U6.11 (GND), U6.14 (GND), U6.2 (GND), U6.36 (GND), U6.37 (GND), U6.38 (GND), U6.39 (GND), U6.40 (GND), U6.41 (GND), U6.42 (GND), U6.43 (GND), U6.44 (GND), U6.45 (GND), U6.46 (GND), U6.47 (GND), U6.48 (GND), U6.49 (GND), U6.50 (GND), U6.51 (GND), U6.52 (GND), U6.53 (GND), U7.5 (VSS), U8.1 (A0), U8.2 (A1), U8.3 (A2), U8.8 (GND), U9.11 (V-)
- new net I2C_SCL: R18.2, U10.8 (SCL), U11.8 (SCL), U12.8 (SCL), U13.8 (SCL), U6.19 (IO5), U7.3 (SCL), U8.14 (SCL)
- new net I2C_SDA: R17.2, U10.7 (SDA), U11.7 (SDA), U12.7 (SDA), U13.7 (SDA), U6.18 (IO4), U7.4 (SDA), U8.15 (SDA)
- new net IO2: R12.2, U6.5 (IO2)
- new net ISO_INA: R1.2, U1.2 (INA)
- new net ISO_INB: R2.2, U1.3 (INB)
- new net LATCH_0V: U16.5 (Q), U7.8 (EVI), U8.4 (P0)
- new net LATCH_OV: U16.9 (Q), U8.5 (P1)
- new net LATCH_RST: R69.2, U16.1 (~{R}), U16.13 (~{R}), U6.21 (IO7)
- new net LED1_A: LED1.2 (A), R16.2
- new net LED2_A: LED2.2 (A), R22.2
- new net LED_ALM: LED2.1 (K), U8.11 (P6)
- new net LED_STAT: LED1.1 (K), R13.2, U6.22 (IO8)
- new net LSET_0V: R67.2, U14.1, U14.13, U14.14, U14.2, U15.1, U15.2, U16.4 (~{S})
- new net LSET_OV: R68.2, U15.14, U16.10 (~{S})
- new net MEAS_15BP: C30.1, R30.2, R40.1, U10.1 (CH1+), U15.8 (-)
- new net MEAS_BA1: C34.1, R34.2, R44.1, U11.1 (CH1+)
- new net MEAS_BA2: C35.1, R35.2, R45.1, U11.3 (CH2+)
- new net MEAS_BA3: C36.1, R36.2, R46.1, U11.11 (CH3+)
- new net MEAS_SIR: C57.1, R84.2, R85.1, U13.13 (CH4+)
- new net MEAS_SW1: C31.1, R31.2, R41.1, U10.3 (CH2+)
- new net MEAS_SW2: C32.1, R32.2, R42.1, U10.11 (CH3+)
- new net MEAS_SW3: C33.1, R33.2, R43.1, U10.13 (CH4+)
- new net MEAS_VBAT: C15.1, R10.1, R9.2, U11.13 (CH4+)
- new net PG_5V: R7.2, R8.1, U8.10 (P5)
- new net RTC_INT: R15.2, U6.16 (IO10), U7.2 (~{INT})
- new net RTC_VB: C20.1, U7.6 (VBACKUP)
- new net SIREN_EN: R83.1, U17.4 (EN), U18.1 (IN), U6.20 (IO6)
- new net SIREN_P: D16.1 (A1), J11.3 (Pin_3), R84.1, U18.3 (OUT)
- new net SNF_SCL: U1.6 (OUTB), U6.12 (IO0)
- new net SNF_SCL_J: JP4.4 (Pin_4), R2.1
- new net SNF_SDA: U1.7 (OUTA), U6.13 (IO1)
- new net SNF_SDA_J: JP4.2 (Pin_2), R1.1
- new net U0RX: J9.4 (Pin_4), U6.30 (RXD0/IO20)
- new net U0TX: J9.3 (Pin_3), U6.31 (TXD0/IO21)
- new net USB_DM: J9.7 (Pin_7), U6.26 (IO18/USB_D-)
- new net USB_DP: J9.8 (Pin_8), U6.27 (IO19/USB_D+)
- new net VBAT: C12.1, C56.1, F5.2, L2.1, Q1.3 (D), R9.1, U17.5 (IN), U4.5 (BAT), U4.8 (FB)
- new net VDIFF1: R60.2, U13.1 (CH1+), U14.5 (+), U14.6 (-), U9.1
- new net VDIFF2: R61.2, U13.3 (CH2+), U14.11 (+), U14.8 (-), U9.7
- new net VDIFF3: R62.2, U13.11 (CH3+), U15.5 (+), U15.6 (-), U9.8
- new net VREF: R57.2, R58.2, R59.2, U13.12 (CH3-), U13.2 (CH1-), U13.4 (CH2-), U9.13 (-), U9.14
- new net VREF_R: C41.1, R64.2, R65.1, U15.10 (-), U9.12 (+)
- new net VSYS: C10.1, C13.1, D6.1 (K), Q1.2 (S), U5.1 (VIN), U5.3 (EN)
- new net VTH_H: R63.2, R64.1, U14.7 (+), U14.9 (+), U15.7 (+), U15.9 (+)
- new net VTH_L: R65.2, R66.1, U14.10 (-), U14.4 (-), U15.4 (-)
- new net Z1_T: D11.1 (A1), J10.1 (Pin_1), R71.1
- new net Z2_T: D12.1 (A1), J10.3 (Pin_3), R72.1
- new net Z3_T: D13.1 (A1), J10.5 (Pin_5), R73.1
- new net Z4_T: D14.1 (A1), J10.7 (Pin_7), R74.1
- new net ZONE1_M: C51.1, R71.2, R75.2, U12.1 (CH1+)
- new net ZONE2_M: C52.1, R72.2, R76.2, U12.3 (CH2+)
- new net ZONE3_M: C53.1, R73.2, R77.2, U12.11 (CH3+)
- new net ZONE4_M: C54.1, R74.2, R78.2, U12.13 (CH4+)
- no-connect marks 0 -> 6
Other:
- note added: "A – ÉCOUTE I2C PASSIVE : cavalier JP4, 1 kΩ série, isolateur unidirectionnel ISO7720 (2 canaux bus → module, aucun canal retour)"
- note added: "B – ALIMENTATION : PTC propre, anti-retour, TVS, abaisseur 15→5 V, chargeur LiFePO4 3,6 V 200 mA (CTN), power-path, LDO 3,3 V"
- note added: "C – MODULE ESP32-C3, RTC RV-3028 (supercondensateur), extension d'E/S TCA9534, débogage"
- note added: "D – MESURES : +15 V amont/aval des PTC (÷16), écart de 0 V (amplis différentiels G = 0,249), ADC MCP3428 x4"
- note added: "E – LATCH SURTENSION : fenêtre ±1 V sur l'écart de 0 V, +15 V > 20 V ; bascule 74HC74 réarmée par GPIO7"
- note added: "F – ALARME : 4 boucles équilibrées (FDL 2 x 4,7 kΩ), clé ARM, sirène 12 V (boost MT3608 + BTS4140N)"
- note added: "N2 « étoile 0 V » – rév. B : carte d'étoile sur rail DIN + module ESP32 espion/alarme Partie bus (change i2c-surge-protection-2026-10-007, Refs #1) : SDA/SCL/+15 V/0 V du BP distribués vers chaque port BA ; par port : cavalier (SDA, SCL, +15 V), PTC puis TVS SMAJ16A. Le 0 V n'est jamais coupé et n'est JAMAIS relié au PE. Module (change n2-esp32-spy-alarm-2026-10-008, essensys-hub/essensys-feature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"
- note removed: "N2 « étoile 0 V » – carte passive sur rail DIN (change OpenSpec i2c-surge-protection-2026-10-007, Refs #1) Bus en étoile : SDA/SCL/+15 V/0 V du BP distribués vers chaque port BA. Par port : cavalier (SDA, SCL, +15 V), PTC puis TVS SMAJ16A sur le +15 V. Le 0 V n'est jamais coupé et n'est JAMAIS relié au PE. Plan 0 V double face, cuivre 2 oz."
- title: N2 étoile 0 V -> N2 étoile 0 V + module ESP32 espion/alarme
